File: ESP32_MicroSD/ESP32_MicroSD.kicad_sch (KiCad schematic)
At the start: 8 parts, among them J1 Conn_01x10_Female, J2 Micro_SD_Card, U1 ESP32-WROOM-32U

Commit message: Update
Parts:
- J2: footprint (none) -> Ariel:Micro_SD_5033981892
Changed lines of the file:
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@@
     (property "Reference" "J2" (id 0) (at 221.615 67.31 0))
     (property "Value" "Micro_SD_Card" (id 1) (at 221.615 69.85 0))
-    (property "Footprint" "" (id 2) (at 250.19 78.74 0)
+    (property "Footprint" "Ariel:Micro_SD_5033981892" (id 2) (at 250.19 78.74 0)
       (effects (font (size 1.27 1.27)) hide)
     )
@@
     )
     (path "/df131e48-1bbb-4d51-8e04-148839fea849"
-      (reference "J2") (unit 1) (value "Micro_SD_Card") (footprint "")
+      (reference "J2") (unit 1) (value "Micro_SD_Card") (footprint "Ariel:Micro_SD_5033981892")
     )
     (path "/6d7a7b7b-8b71-4eb4-944c-7eca1647fd54"

Commit message: update
Parts:
- added C2: 100u, Capacitor_SMD:CP_Elec_4x5.7, symbol Device:C_Polarized_Small
- added D1: LED, symbol Device:LED
- added JP1: Jumper_2_Open, symbol Jumper:Jumper_2_Open
- added R5: 10K, Resistor_SMD:R_0805_2012Metric, symbol Device:R_US
- added SW1: On, Button_Switch_SMD:SW_SPDT_PCM12, symbol Switch:SW_Push_SPDT
Connections:
- net +3V3: now also U1.2 (VDD), C2.1, SW1.2 (B)
- net GND: now also C2.2, JP1.1 (A), R5.2
- net at J1.7 (Pin_7): now also U1.3 (EN), JP1.2 (B)
- net at U1.7 (IO35): now also D1.2 (A)
- new net: J1.1 (Pin_1), SW1.1 (A)
- new net: D1.1 (K), R5.1
- no-connect marks 32 -> 30

Commit message: update
Parts:
- D1: footprint (none) -> LED_SMD:LED_0805_2012Metric
Changed lines of the file:
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@@
     (property "Reference" "D1" (id 0) (at 146.3675 106.68 0))
     (property "Value" "LED" (id 1) (at 146.3675 109.22 0))
-    (property "Footprint" "" (id 2) (at 144.78 114.3 0)
+    (property "Footprint" "LED_SMD:LED_0805_2012Metric" (id 2) (at 144.78 114.3 0)
       (effects (font (size 1.27 1.27)) hide)
     )
@@
     )
     (path "/c44472a6-5859-4bba-8e92-30fe02165afa"
-      (reference "D1") (unit 1) (value "LED") (footprint "")
+      (reference "D1") (unit 1) (value "LED") (footprint "LED_SMD:LED_0805_2012Metric")
     )
     (path "/3325906f-07a8-47c3-9541-eca4478826f1"

Commit message: acomodar pinHeader
Parts:
- JP1: footprint (none) -> Jumper:SolderJumper-2_P1.3mm_Open_Pad1.0x1.5mm
Connections:
- net +3V3: now also SW1.1 (A); no longer SW1.2 (B)
- net GND: now also J1.10 (Pin_10)
- net at J1.1 (Pin_1): now also SW1.2 (B); no longer SW1.1 (A)
- no-connect marks 30 -> 29
Other:
- moved on the sheet: SW1
Changed lines of the file:
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@@
   (no_connect (at 50.8 92.71))
   (no_connect (at 50.8 95.25))
-  (no_connect (at 50.8 97.79))
   (no_connect (at 50.8 82.55))
   (no_connect (at 50.8 77.47))
@@
     (stroke (width 0) (type default) (color 0 0 0 0))
   )
-  (wire (pts (xy 33.02 52.07) (xy 33.02 46.99))
-    (stroke (width 0) (type default) (color 0 0 0 0))
-  )
   (wire (pts (xy 118.11 40.64) (xy 118.11 46.99))
     (stroke (width 0) (type default) (color 0 0 0 0))
@@
     (stroke (width 0) (type default) (color 0 0 0 0))
   )
+  (wire (pts (xy 33.02 46.99) (xy 33.02 53.34))
+    (stroke (width 0) (type default) (color 0 0 0 0))
+  )
   (wire (pts (xy 35.56 74.93) (xy 50.8 74.93))
     (stroke (width 0) (type default) (color 0 0 0 0))
@@
     (stroke (width 0) (type default) (color 0 0 0 0))
   )
+  (wire (pts (xy 35.56 63.5) (xy 35.56 74.93))
+    (stroke (width 0) (type default) (color 0 0 0 0))
+  )
   (wire (pts (xy 167.64 62.23) (xy 179.07 62.23))
     (stroke (width 0) (type default) (color 0 0 0 0))
@@
     (stroke (width 0) (type default) (color 0 0 0 0))
   )
+  (wire (pts (xy 48.26 97.79) (xy 50.8 97.79))
+    (stroke (width 0) (type default) (color 0 0 0 0))
+  )
   (wire (pts (xy 133.35 114.3) (xy 140.97 114.3))
-    (stroke (width 0) (type default) (color 0 0 0 0))
-  )
-  (wire (pts (xy 35.56 62.23) (xy 35.56 74.93))
     (stroke (width 0) (type default) (color 0 0 0 0))
   )
@@
     (property "Reference" "JP1" (id 0) (at 74.93 49.53 0))
     (property "Value" "Jumper_2_Open" (id 1) (at 74.93 52.07 0))
-    (property "Footprint" "" (id 2) (at 74.93 55.88 0)
+    (property "Footprint" "Jumper:SolderJumper-2_P1.3mm_Open_Pad1.0x1.5mm" (id 2) (at 74.93 55.88 0)
       (effects (font (size 1.27 1.27)) hide)
     )
@@
     )
     (property "Datasheet" "" (id 3) (at 53.34 60.96 0)
+      (effects (font (size 1.27 1.27)) hide)
+    )
+    (pin "1")
+  )
+  (symbol (lib_id "power:GND") (at 48.26 97.79 0) (unit 1)
+    (in_bom yes) (on_board yes)
+    (property "Reference" "#PWR0108" (id 0) (at 48.26 104.14 0)
+      (effects (font (size 1.27 1.27)) hide)
+    )
+    (property "Value" "GND" (id 1) (at 43.18 97.79 0))
+    (property "Footprint" "" (id 2) (at 48.26 97.79 0)
+      (effects (font (size 1.27 1.27)) hide)
+    )
+    (property "Datasheet" "" (id 3) (at 48.26 97.79 0)
       (effects (font (size 1.27 1.27)) hide)
     )
@@
     (pin "1")
   )
-  (symbol (lib_id "Switch:SW_Push_SPDT") (at 33.02 57.15 270) (unit 1)
-    (in_bom yes) (on_board yes) (fields_autoplaced)
-    (property "Reference" "SW1" (id 0) (at 36.83 55.8799 90)
-      (effects (font (size 1.27 1.27)) (justify left))
-    )
-    (property "Value" "On" (id 1) (at 36.83 58.4199 90)
-      (effects (font (size 1.27 1.27)) (justify left))
-    )
-    (property "Footprint" "Button_Switch_SMD:SW_SPDT_PCM12" (id 2) (at 33.02 57.15 0)
-      (effects (font (size 1.27 1.27)) hide)
-    )
-    (property "Datasheet" "~" (id 3) (at 33.02 57.15 0)
+  (symbol (lib_id "Switch:SW_Push_SPDT") (at 35.56 58.42 90) (unit 1)
+    (in_bom yes) (on_board yes) (fields_autoplaced)
+    (property "Reference" "SW1" (id 0) (at 39.37 57.1499 90)
+      (effects (font (size 1.27 1.27)) (justify right))
+    )
+    (property "Value" "On" (id 1) (at 39.37 59.6899 90)
+      (effects (font (size 1.27 1.27)) (justify right))
+    )
+    (property "Footprint" "Button_Switch_SMD:SW_SPDT_PCM12" (id 2) (at 35.56 58.42 0)
+      (effects (font (size 1.27 1.27)) hide)
+    )
+    (property "Datasheet" "~" (id 3) (at 35.56 58.42 0)
       (effects (font (size 1.27 1.27)) hide)
     )
@@
       (reference "#PWR0107") (unit 1) (value "+3.3V") (footprint "")
     )
+    (path "/d59ae9b4-0090-4b31-a49c-cffd4f10dfde"
+      (reference "#PWR0108") (unit 1) (value "GND") (footprint "")
+    )
     (path "/df8ed8d2-6b17-4e6d-8753-58bf3b50175f"
       (reference "C1") (unit 1) (value "100n") (footprint "Capacitor_SMD:C_0805_2012Metric")
@@
     )
     (path "/7c1cc0d3-5f9e-46fd-9e67-64f1904f0fd5"
-      (reference "JP1") (unit 1) (value "Jumper_2_Open") (footprint "")
+      (reference "JP1") (unit 1) (value "Jumper_2_Open") (footprint "Jumper:SolderJumper-2_P1.3mm_Open_Pad1.0x1.5mm")
     )
     (path "/6d7a7b7b-8b71-4eb4-944c-7eca1647fd54"

Commit message: Fix J1
Parts:
- removed C2: 100u, Capacitor_SMD:CP_Elec_4x5.7, symbol Device:C_Polarized_Small
- added C2: 10u, Capacitor_SMD:C_0805_2012Metric, symbol Device:C_Small
- R5: value 10K -> 68R
Connections:
- net +3V3: now also C2.1
- net GND: now also J1.11 (Pin_11), C2.2; no longer J1.10 (Pin_10), J1.3 (Pin_3)
- net RX: now also J1.13 (Pin_13); no longer J1.5 (Pin_5)
- net TX: now also J1.14 (Pin_14); no longer J1.6 (Pin_6)
- net at SW1.2 (B): now also J1.9 (Pin_9); no longer J1.1 (Pin_1)
- net at JP1.2 (B), U1.3 (EN): no longer J1.7 (Pin_7)
- no-connect marks 29 -> 35
Changed lines of the file:
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@@
   (junction (at 194.31 81.28) (diameter 0) (color 0 0 0 0)
   )
-  (junction (at 80.01 55.88) (diameter 0) (color 0 0 0 0)
-  )
   (junction (at 167.64 91.44) (diameter 0) (color 0 0 0 0)
   )
@@
   (junction (at 179.07 62.23) (diameter 0) (color 0 0 0 0)
   )
+  (no_connect (at 38.1 53.34))
+  (no_connect (at 241.3 101.6))
+  (no_connect (at 198.12 96.52))
+  (no_connect (at 198.12 78.74))
   (no_connect (at 50.8 92.71))
   (no_connect (at 50.8 95.25))
@@
   (no_connect (at 102.87 88.9))
   (no_connect (at 102.87 86.36))
+  (no_connect (at 50.8 97.79))
+  (no_connect (at 50.8 90.17))
   (no_connect (at 133.35 73.66))
   (no_connect (at 133.35 71.12))
@@
     (stroke (width 0) (type default) (color 0 0 0 0))
   )
-  (wire (pts (xy 45.72 90.17) (xy 45.72 109.22))
-    (stroke (width 0) (type default) (color 0 0 0 0))
-  )
   (wire (pts (xy 194.31 81.28) (xy 198.12 81.28))
     (stroke (width 0) (type default) (color 0 0 0 0))
@@
     (stroke (width 0) (type default) (color 0 0 0 0))
   )
-  (wire (pts (xy 50.8 90.17) (xy 45.72 90.17))
-    (stroke (width 0) (type default) (color 0 0 0 0))
-  )
   (wire (pts (xy 118.11 40.64) (xy 118.11 46.99))
     (stroke (width 0) (type default) (color 0 0 0 0))
@@
     (stroke (width 0) (type default) (color 0 0 0 0))
   )
-  (wire (pts (xy 80.01 109.22) (xy 80.01 55.88))
-    (stroke (width 0) (type default) (color 0 0 0 0))
-  )
   (wire (pts (xy 184.15 72.39) (xy 184.15 88.9))
     (stroke (width 0) (type default) (color 0 0 0 0))
@@
     (stroke (width 0) (type default) (color 0 0 0 0))
   )
-  (wire (pts (xy 45.72 109.22) (xy 80.01 109.22))
-    (stroke (width 0) (type default) (color 0 0 0 0))
-  )
   (wire (pts (xy 179.07 93.98) (xy 198.12 93.98))
     (stroke (width 0) (type default) (color 0 0 0 0))
@@
   )
   (wire (pts (xy 198.12 86.36) (xy 167.64 86.36))
-    (stroke (width 0) (type default) (color 0 0 0 0))
-  )
-  (wire (pts (xy 48.26 97.79) (xy 50.8 97.79))
     (stroke (width 0) (type default) (color 0 0 0 0))
   )
@@
     (pin "1")
   )
+  (symbol (lib_id "Device:C_Small") (at 53.34 52.07 0) (unit 1)
+    (in_bom yes) (on_board yes)
+    (property "Reference" "C2" (id 0) (at 46.99 52.07 0)
+      (effects (font (size 1.27 1.27)) (justify left))
+    )
+    (property "Value" "10u" (id 1) (at 46.99 54.61 0)
+      (effects (font (size 1.27 1.27)) (justify left))
+    )
+    (property "Footprint" "Capacitor_SMD:C_0805_2012Metric" (id 2) (at 53.34 52.07 0)
+      (effects (font (size 1.27 1.27)) hide)
+    )
+    (property "Datasheet" "~" (id 3) (at 53.34 52.07 0)
+      (effects (font (size 1.27 1.27)) hide)
+    )
+    (pin "1")
+    (pin "2")
+  )
   (symbol (lib_id "Device:R_US") (at 184.15 68.58 0) (unit 1)
     (in_bom yes) (on_board yes)
@@
       (effects (font (size 1.27 1.27)) hide)
     )
-    (pin "1")
+    (pin "9")
+    (pin "18")
     (pin "10")
-    (pin "2")
-    (pin "3")
-    (pin "4")
-    (pin "5")
-    (pin "6")
-    (pin "7")
-    (pin "8")
-    (pin "9")
-  )
-  (symbol (lib_id "Device:C_Polarized_Small") (at 53.34 52.07 0) (unit 1)
-    (in_bom yes) (on_board yes)
-    (property "Reference" "C2" (id 0) (at 55.88 50.2538 0)
-      (effects (font (size 1.27 1.27)) (justify left))
-    )
-    (property "Value" "100u" (id 1) (at 46.99 49.53 0)
-      (effects (font (size 1.27 1.27)) (justify left))
-    )
-    (property "Footprint" "Capacitor_SMD:CP_Elec_4x5.7" (id 2) (at 53.34 52.07 0)
-      (effects (font (size 1.27 1.27)) hide)
-    )
-    (property "Datasheet" "~" (id 3) (at 53.34 52.07 0)
-      (effects (font (size 1.27 1.27)) hide)
-    )
-    (pin "1")
-    (pin "2")
+    (pin "11")
+    (pin "12")
+    (pin "13")
+    (pin "14")
+    (pin "15")
+    (pin "16")
+    (pin "17")
   )
   (symbol (lib_id "power:+3.3V") (at 184.15 54.61 0) (unit 1)
@@
       (effects (font (size 1.27 1.27)) (justify left))
     )
-    (property "Value" "10K" (id 1) (at 148.59 121.92 0)
+    (property "Value" "68R" (id 1) (at 148.59 121.92 0)
       (effects (font (size 1.27 1.27)) (justify left))
     )
@@
     )
     (property "Datasheet" "" (id 3) (at 53.34 60.96 0)
-      (effects (font (size 1.27 1.27)) hide)
-    )
-    (pin "1")
-  )
-  (symbol (lib_id "power:GND") (at 48.26 97.79 0) (unit 1)
-    (in_bom yes) (on_board yes)
-    (property "Reference" "#PWR0108" (id 0) (at 48.26 104.14 0)
-      (effects (font (size 1.27 1.27)) hide)
-    )
-    (property "Value" "GND" (id 1) (at 43.18 97.79 0))
-    (property "Footprint" "" (id 2) (at 48.26 97.79 0)
-      (effects (font (size 1.27 1.27)) hide)
-    )
-    (property "Datasheet" "" (id 3) (at 48.26 97.79 0)
       (effects (font (size 1.27 1.27)) hide)
     )
@@
       (reference "#PWR0107") (unit 1) (value "+3.3V") (footprint "")
     )
-    (path "/d59ae9b4-0090-4b31-a49c-cffd4f10dfde"
-      (reference "#PWR0108") (unit 1) (value "GND") (footprint "")
-    )
     (path "/df8ed8d2-6b17-4e6d-8753-58bf3b50175f"
       (reference "C1") (unit 1) (value "100n") (footprint "Capacitor_SMD:C_0805_2012Metric")
     )
-    (path "/3faed274-51d7-4d4b-b396-045ef95a516d"
-      (reference "C2") (unit 1) (value "100u") (footprint "Capacitor_SMD:CP_Elec_4x5.7")
+    (path "/205b61c0-f602-4203-af98-d178169357d8"
+      (reference "C2") (unit 1) (value "10u") (footprint "Capacitor_SMD:C_0805_2012Metric")
     )
     (path "/c44472a6-5859-4bba-8e92-30fe02165afa"
@@
     )
     (path "/75c2f375-a96c-4783-bb5b-4ae9ca26228a"
-      (reference "R5") (unit 1) (value "10K") (footprint "Resistor_SMD:R_0805_2012Metric")
+      (reference "R5") (unit 1) (value "68R") (footprint "Resistor_SMD:R_0805_2012Metric")
     )
     (path "/f82608ac-609f-4c91-ab78-5ac8ba0d40c9"
